File: Eagle/Arduino-DRA818V-TX/Arduino-DRA818V-TX.sch (EAGLE design)
At the start: 23 parts, among them M1 ARDUINO_R3_ICSP, X1 SMA, X2 SMA

Commit message: Using 0805 SMDs
Parts:
- ANT1, ANT2: value SMA -> 50 Z
- C1, C10, C2, C5, C6, C7, C8: device resistor:C-EUC1206 -> resistor:C-EUC0805
- C3, C9: value 1u -> 100n; device resistor:C-EUC1206 -> resistor:C-EUC0805
- C4: value 100n -> 1u; device resistor:C-EUC1206 -> resistor:C-EUC0805
- GPS: value (none) -> + TX RX GND
- R1: device resistor:R-US_R1206 -> resistor:R-US_R0805
- R2: value 1k -> 560; device resistor:R-US_R1206 -> resistor:R-US_R0805
- R3: value 560 -> 5k6; device resistor:R-US_R1206 -> resistor:R-US_R0805
- renumbered JP1 to GPS, X1 to ANT1, X2 to ANT2
Connections:
- net +5V: now also C4.1; no longer C10.1
- net AF_NORM: now also C10.2; no longer C9.2
- net GND: now also C9.2; no longer C10.2
- net LED_BUILTIN: now also R2.2; no longer R3.2
- net N$7: now also C5.1, R3.1; no longer C6.1, R2.1
- net N$8: now also R2.1; no longer R3.1
- net N$9: now also C10.1; no longer C8.1
- net PD: now also C7.1; no longer C4.1
- net POW: now also C8.1; no longer C5.1
- net PTT: now also R3.2; no longer R2.2
- net PTT_SW: now also C6.1; no longer C7.1
Other:
- moved on the sheet: C1, C10, C2, C3, C4, C5, C6, C7, C8, C9, R2, R3
